File: ecad/reminder-mainboard/reminder-mainboard.sch (KiCad schematic (older format))
At the start: 27 parts, among them J1 USB_B_Micro, J2 MOLEX SL 1x5, J3 Conn_01x03_Male, J4 22-03-5065, Q1 2N3904, SW1 SW_SPDT, SW2 SW_Push, SW3 SW_Push, U1 LM1117-3.3, U2 QRD1113GR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

Commit message: Readied for adding separate usb chip
Parts:
- added C?: 10uF, Capacitor_Tantalum_SMD:CP_EIA-3528-21_Kemet-B, symbol Device:C_Small
- added U?: MCP2221, Package_SO:TSSOP-14_4.4x5mm_P0.65mm, symbol MCP2221:MCP2221
- U3: symbol MCU_ST_STM32F0:STM32F042F4Px -> MCU_ST_STM32F0:STM32F030F4Px
Connections:
- net labels added: USB_RST
- wire segments 93 -> 101
- no-connect marks 7 -> 12
Other:
- note added: "USB Interface"
- moved on the sheet: C1, C2, U1
Changed lines of the file:
@@
 $EndComp
 Wire Wire Line
-	4000 1950 4000 1850
-Wire Wire Line
-	3100 1950 3100 1850
-Wire Wire Line
-	3100 1600 3250 1600
-Wire Wire Line
-	3100 1650 3100 1600
-Wire Wire Line
-	4000 1600 4100 1600
-Wire Wire Line
-	4000 1650 4000 1600
-Connection ~ 4000 1600
-Wire Wire Line
-	3850 1600 4000 1600
-Connection ~ 3100 1600
-Wire Wire Line
-	3000 1600 3100 1600
+	5950 1950 5950 1850
+Wire Wire Line
+	5050 1950 5050 1850
+Wire Wire Line
+	5050 1600 5200 1600
+Wire Wire Line
+	5050 1650 5050 1600
+Wire Wire Line
+	5950 1600 6050 1600
+Wire Wire Line
+	5950 1650 5950 1600
+Connection ~ 5950 1600
+Wire Wire Line
+	5800 1600 5950 1600
+Connection ~ 5050 1600
+Wire Wire Line
+	4950 1600 5050 1600
 Wire Wire Line
 	1900 1750 2000 1750
@@
 	2000 1300 2000 1450
 Wire Wire Line
-	4100 1600 4100 1500
-Wire Wire Line
-	4000 1950 3550 1950
-Wire Wire Line
-	3550 1950 3550 2050
-Wire Wire Line
-	3550 1950 3550 1900
-Connection ~ 3550 1950
-Wire Wire Line
-	3100 1950 3550 1950
-Wire Wire Line
-	3000 1500 3000 1600
+	6050 1600 6050 1500
+Wire Wire Line
+	5950 1950 5500 1950
+Wire Wire Line
+	5500 1950 5500 2050
+Wire Wire Line
+	5500 1950 5500 1900
+Connection ~ 5500 1950
+Wire Wire Line
+	5050 1950 5500 1950
+Wire Wire Line
+	4950 1500 4950 1600
 $Comp
 L power:+5V #PWR07
 U 1 1 604A7B58
-P 3000 1500
-F 0 "#PWR07" H 3000 1350 50  0001 C CNN
-F 1 "+5V" H 3015 1673 50  0000 C CNN
-F 2 "" H 3000 1500 50  0001 C CNN
-F 3 "" H 3000 1500 50  0001 C CNN
-	1    3000 1500
+P 4950 1500
+F 0 "#PWR07" H 4950 1350 50  0001 C CNN
+F 1 "+5V" H 4965 1673 50  0000 C CNN
+F 2 "" H 4950 1500 50  0001 C CNN
+F 3 "" H 4950 1500 50  0001 C CNN
+	1    4950 1500
 	1    0    0    -1
 $EndComp
@@
 L Device:C_Small C1
 U 1 1 604A6438
-P 3100 1750
-F 0 "C1" H 3009 1796 50  0000 R CNN
-F 1 "10uF" H 3009 1705 50  0000 R CNN
-F 2 "Capacitor_Tantalum_SMD:CP_EIA-6032-28_Kemet-C" H 3100 1750 50  0001 C CNN
-F 3 "https://datasheet.lcsc.com/szlcsc/KEMET-T491C106K025AT_C116748.pdf" H 3100 1750 50  0001 C CNN
-F 4 "T491C106K025AT" H 3100 1750 50  0001 C CNN "Mfg PN"
-F 5 "KEMET" H 3100 1750 50  0001 C CNN "Mfg"
-	1    3100 1750
-	1    0    0    -1
-$EndComp
-Text Notes 2950 900  0    79   ~ 16
+P 5050 1750
+F 0 "C1" H 4959 1796 50  0000 R CNN
+F 1 "10uF" H 4959 1705 50  0000 R CNN
+F 2 "Capacitor_Tantalum_SMD:CP_EIA-6032-28_Kemet-C" H 5050 1750 50  0001 C CNN
+F 3 "https://datasheet.lcsc.com/szlcsc/KEMET-T491C106K025AT_C116748.pdf" H 5050 1750 50  0001 C CNN
+F 4 "T491C106K025AT" H 5050 1750 50  0001 C CNN "Mfg PN"
+F 5 "KEMET" H 5050 1750 50  0001 C CNN "Mfg"
+	1    5050 1750
+	1    0    0    -1
+$EndComp
+Text Notes 4900 900  0    79   ~ 16
 DC Power Conversion
 Text Notes 1400 900  0    79   ~ 16
@@
 L power:GND #PWR08
 U 1 1 60487D66
-P 3550 2050
-F 0 "#PWR08" H 3550 1800 50  0001 C CNN
-F 1 "GND" H 3555 1877 50  0000 C CNN
-F 2 "" H 3550 2050 50  0001 C CNN
-F 3 "" H 3550 2050 50  0001 C CNN
-	1    3550 2050
+P 5500 2050
+F 0 "#PWR08" H 5500 1800 50  0001 C CNN
+F 1 "GND" H 5505 1877 50  0000 C CNN
+F 2 "" H 5500 2050 50  0001 C CNN
+F 3 "" H 5500 2050 50  0001 C CNN
+	1    5500 2050
 	1    0    0    -1
 $EndComp
@@
 L power:+3.3V #PWR011
 U 1 1 60461D21
-P 4100 1500
-F 0 "#PWR011" H 4100 1350 50  0001 C CNN
-F 1 "+3.3V" H 4115 1673 50  0000 C CNN
-F 2 "" H 4100 1500 50  0001 C CNN
-F 3 "" H 4100 1500 50  0001 C CNN
-	1    4100 1500
+P 6050 1500
+F 0 "#PWR011" H 6050 1350 50  0001 C CNN
+F 1 "+3.3V" H 6065 1673 50  0000 C CNN
+F 2 "" H 6050 1500 50  0001 C CNN
+F 3 "" H 6050 1500 50  0001 C CNN
+	1    6050 1500
 	1    0    0    -1
 $EndComp
@@
 L Regulator_Linear:LM1117-3.3 U1
 U 1 1 603E6E60
-P 3550 1600
-F 0 "U1" H 3550 1842 50  0000 C CNN
-F 1 "LM1117-3.3" H 3550 1751 50  0000 C CNN
-F 2 "Package_TO_SOT_SMD:SOT-223-3_TabPin2" H 3550 1600 50  0001 C CNN
-F 3 "https://datasheet.lcsc.com/szlcsc/Texas-Instruments-TI-LM1117IMPX-3-3-NOPB_C23984.pdf" H 3550 1600 50  0001 C CNN
-F 4 "Texas Instruments" H 3550 1600 50  0001 C CNN "Mfg"
-F 5 "LM1117IMPX-3.3/NOPB" H 3550 1600 50  0001 C CNN "Mfg PN"
-	1    3550 1600
+P 5500 1600
+F 0 "U1" H 5500 1842 50  0000 C CNN
+F 1 "LM1117-3.3" H 5500 1751 50  0000 C CNN
+F 2 "Package_TO_SOT_SMD:SOT-223-3_TabPin2" H 5500 1600 50  0001 C CNN
+F 3 "https://datasheet.lcsc.com/szlcsc/Texas-Instruments-TI-LM1117IMPX-3-3-NOPB_C23984.pdf" H 5500 1600 50  0001 C CNN
+F 4 "Texas Instruments" H 5500 1600 50  0001 C CNN "Mfg"
+F 5 "LM1117IMPX-3.3/NOPB" H 5500 1600 50  0001 C CNN "Mfg PN"
+	1    5500 1600
 	1    0    0    -1
 $EndComp
@@
 Text Label 9750 1950 0    39   ~ 0
 LED_R
-NoConn ~ 9550 1850
 $Comp
 L power:GND #PWR024
@@
 Text Label 9750 2850 0    39   ~ 0
 SWDIO
-Text Label 9750 2750 0    39   ~ 0
-USB_P
-Text Label 9750 2650 0    39   ~ 0
-USB_M
 Text Label 7100 1850 2    39   ~ 0
 NRST
@@
 NoConn ~ 8350 2850
 $Comp
-L MCU_ST_STM32F0:STM32F042F4Px U3
+L MCU_ST_STM32F0:STM32F030F4Px U3
 U 1 1 603DE65E
 P 8950 2350
@@
 F 1 "STM32F042F4Px" H 9250 1400 50  0000 C CNN
 F 2 "Package_SO:TSSOP-20_4.4x6.5mm_P0.65mm" H 8450 1650 50  0001 R CNN
-F 3 "http://www.st.com/st-web-ui/static/active/en/resource/technical/document/datasheet/DM00105814.pdf" H 8950 2350 50  0001 C CNN
+F 3 "https://datasheet.lcsc.com/szlcsc/STMicroelectronics-STM32F205RET6_C66278.pdf" H 8950 2350 50  0001 C CNN
 	1    8950 2350
 	1    0    0    -1
@@
 $EndComp
 Wire Wire Line
-	10000 1600 10000 1650
-Wire Wire Line
 	8750 1400 8750 1650
 Wire Wire Line
@@
 L power:GND #PWR027
 U 1 1 6056EBB5
-P 10000 1650
-F 0 "#PWR027" H 10000 1400 50  0001 C CNN
-F 1 "GND" H 10005 1477 50  0000 C CNN
-F 2 "" H 10000 1650 50  0001 C CNN
-F 3 "" H 10000 1650 50  0001 C CNN
-	1    10000 1650
+P 10000 1600
+F 0 "#PWR027" H 10000 1350 50  0001 C CNN
+F 1 "GND" H 10150 1500 50  0000 C CNN
+F 2 "" H 10000 1600 50  0001 C CNN
+F 3 "" H 10000 1600 50  0001 C CNN
+	1    10000 1600
 	1    0    0    -1
 $EndComp
@@
 L Device:C_Small C2
 U 1 1 604AE413
-P 4000 1750
-F 0 "C2" H 4092 1796 50  0000 L CNN
-F 1 "100uF" H 4092 1705 50  0000 L CNN
-F 2 "Capacitor_Tantalum_SMD:CP_EIA-3528-21_Kemet-B" H 4000 1750 50  0001 C CNN
-F 3 "https://datasheet.lcsc.com/szlcsc/AVX-TAJB107K006RNJ_C16133.pdf" H 4000 1750 50  0001 C CNN
-F 4 "TAJB107K006RNJ" H 4000 1750 50  0001 C CNN "Mfg PN"
-F 5 "AVX" H 4000 1750 50  0001 C CNN "Mfg"
-	1    4000 1750
-	1    0    0    -1
-$EndComp
+P 5950 1750
+F 0 "C2" H 6042 1796 50  0000 L CNN
+F 1 "100uF" H 6042 1705 50  0000 L CNN
+F 2 "Capacitor_Tantalum_SMD:CP_EIA-3528-21_Kemet-B" H 5950 1750 50  0001 C CNN
+F 3 "https://datasheet.lcsc.com/szlcsc/AVX-TAJB107K006RNJ_C16133.pdf" H 5950 1750 50  0001 C CNN
+F 4 "TAJB107K006RNJ" H 5950 1750 50  0001 C CNN "Mfg PN"
+F 5 "AVX" H 5950 1750 50  0001 C CNN "Mfg"
+	1    5950 1750
+	1    0    0    -1
+$EndComp
+Text Notes 3050 900  0    79   ~ 16
+USB Interface
+$Comp
+L MCP2221:MCP2221 U?
+U 1 1 6053D612
+P 3300 1300
+F 0 "U?" H 3475 1375 50  0000 C CNN
+F 1 "MCP2221" H 3475 1284 50  0000 C CNN
+F 2 "Package_SO:TSSOP-14_4.4x5mm_P0.65mm" H 3300 1300 50  0001 C CNN
+F 3 "https://www.mouser.com/datasheet/2/268/20005292A-357587.pdf" H 3300 1300 50  0001 C CNN
+	1    3300 1300
+	1    0    0    -1
+$EndComp
+Text Label 9750 2750 0    39   ~ 0
+USB_P
+Text Label 9750 2650 0    39   ~ 0
+USB_M
+$Comp
+L power:+3.3V #PWR?
+U 1 1 6054B3B5
+P 3000 1350
+F 0 "#PWR?" H 3000 1200 50  0001 C CNN
+F 1 "+3.3V" H 3015 1523 50  0000 C CNN
+F 2 "" H 3000 1350 50  0001 C CNN
+F 3 "" H 3000 1350 50  0001 C CNN
+	1    3000 1350
+	1    0    0    -1
+$EndComp
+Text Label 9750 1850 0    39   ~ 0
+USB_RST
+Wire Wire Line
+	9750 1850 9550 1850
+Wire Wire Line
+	3000 1350 3000 1450
+Wire Wire Line
+	3000 1450 3100 1450
+NoConn ~ 3100 1550
+NoConn ~ 3100 1650
+NoConn ~ 3100 2050
+NoConn ~ 3850 2050
+Text Label 2900 1750 2    50   ~ 0
+USB_RST
+Wire Wire Line
+	2900 1750 3100 1750
+NoConn ~ 3850 1850
+NoConn ~ 3850 1950
+$Comp
+L Device:C_Small C?
+U 1 1 60598A81
+P 4100 1850
+F 0 "C?" H 4192 1896 50  0000 L CNN
+F 1 "10uF" H 4192 1805 50  0000 L CNN
+F 2 "Capacitor_Tantalum_SMD:CP_EIA-3528-21_Kemet-B" H 4100 1850 50  0001 C CNN
+F 3 "https://datasheet.lcsc.com/szlcsc/AVX-TAJB106M025RNJ_C8018.pdf" H 4100 1850 50  0001 C CNN
+F 4 "AVX" H 4100 1850 50  0001 C CNN "Mfg"
+F 5 "TAJB106M025RNJ" H 4100 1850 50  0001 C CNN "Mfg PN"
+	1    4100 1850
+	1    0    0    -1
+$EndComp
+Wire Wire Line
+	4100 1750 3850 1750
+$Comp
+L power:GND #PWR?
+U 1 1 6059CD1A
+P 4100 1950
+F 0 "#PWR?" H 4100 1700 50  0001 C CNN
+F 1 "GND" H 4105 1777 50  0000 C CNN
+F 2 "" H 4100 1950 50  0001 C CNN
+F 3 "" H 4100 1950 50  0001 C CNN
+	1    4100 1950
+	1    0    0    -1
+$EndComp
+Text Label 4000 1550 0    50   ~ 0
+USB_P
+Text Label 4000 1650 0    50   ~ 0
+USB_M
+Wire Wire Line
+	4000 1650 3850 1650
+Wire Wire Line
+	4000 1550 3850 1550
+$Comp
+L power:GND #PWR?
+U 1 1 605A4759
+P 4550 1950
+F 0 "#PWR?" H 4550 1700 50  0001 C CNN
+F 1 "GND" H 4555 1777 50  0000 C CNN
+F 2 "" H 4550 1950 50  0001 C CNN
+F 3 "" H 4550 1950 50  0001 C CNN
+	1    4550 1950
+	1    0    0    -1
+$EndComp
+Wire Wire Line
+	3850 1450 4550 1450
+Wire Wire Line
+	4550 1450 4550 1950
 $EndSCHEMATC

Commit message: Started work on RPI-hat version
Parts:
- removed BZ1: Buzzer, Connector_Molex:Molex_SL_171971-0002_1x02_P2.54mm_Vertical, symbol Device:Buzzer
- removed C1: 10uF, Capacitor_Tantalum_SMD:CP_EIA-6032-28_Kemet-C, symbol Device:C_Small
- removed C2: 100uF, Capacitor_Tantalum_SMD:CP_EIA-3528-21_Kemet-B, symbol Device:C_Small
- removed C3, C4, C5: 100nF, Capacitor_SMD:C_0805_2012Metric, symbol Device:C_Small
- removed C6, C?: 10uF, Capacitor_Tantalum_SMD:CP_EIA-3528-21_Kemet-B, symbol Device:C_Small
- removed J1: USB_B_Micro, Connector_Molex:Molex_SL_171971-0006_1x06_P2.54mm_Vertical, symbol Connector:USB_B_Micro
- removed J2: MOLEX SL 1x5, Connector_Molex:Molex_SL_171971-0005_1x05_P2.54mm_Vertical, symbol Connector_Generic:Conn_01x05
- removed J3: Conn_01x03_Male, Connector_PinHeader_2.54mm:PinHeader_1x03_P2.54mm_Vertical, symbol Connector:Conn_01x03_Male
- removed J4: 22-03-5065, Connector_Molex:Molex_SPOX_5267-06A_1x06_P2.50mm_Vertical, symbol Connector:Conn_01x06_Male
- removed R4: 160, Resistor_SMD:R_0603_1608Metric, symbol Device:R_Small_US
- removed R5, R6, R7: 10k, Resistor_SMD:R_0603_1608Metric, symbol Device:R_Small_US
- removed SW1: SW_SPDT, Connector_Molex:Molex_SL_171971-0003_1x03_P2.54mm_Vertical, symbol Switch:SW_SPDT
- removed SW2: SW_Push, Connector_Molex:Molex_SL_171971-0002_1x02_P2.54mm_Vertical, symbol Switch:SW_Push
- removed SW3: SW_Push, jlcpcb:TACT_SWITCH_TS-1187A-X-X-X, symbol Switch:SW_Push
- removed U1: LM1117-3.3, Package_TO_SOT_SMD:SOT-223-3_TabPin2, symbol Regulator_Linear:LM1117-3.3
- removed U2: QRD1113GR, OptoDevice:Everlight_ITR8307F43, symbol SENSOR_PROX_QRD:QRD1113GR
- removed U3: STM32F042F4Px, Package_SO:TSSOP-20_4.4x6.5mm_P0.65mm, symbol MCU_ST_STM32F0:STM32F030F4Px
- removed U?: MCP2221, Package_SO:TSSOP-14_4.4x5mm_P0.65mm, symbol MCP2221:MCP2221
- added H? (x2): MountingHole, MountingHole:MountingHole_2.7mm_M2.5_Pad, symbol Mechanical:MountingHole
- added J? (x6): Conn_01x04, symbol Connector:Conn_01x04_Male
- added J?: Raspberry_Pi_2_3, symbol Connector:Raspberry_Pi_2_3
- added J? (x3): Conn_01x02_Male, symbol Connector:Conn_01x02_Male
- added J? (x3): Conn_01x03_Male, symbol Connector:Conn_01x03_Male
Connections:
- net labels removed: LED_B, LED_G, LED_R, NRST, SENSOR, SWCLK, SWDIO, USB_M, USB_P, USB_RST
- wire segments 101 -> 90
- no-connect marks 12 -> 0
Other:
- note added: "5V Entry"
- note added: "GPIO Expansion"
- note added: "LED Board Connectors\n"
- note added: "Prox Sensor Connectors\n"
- note removed: "ARM MCU"
- note removed: "DC Power Conversion"
- note removed: "LED Board Conn.\n"
- note removed: "Prox Sensor"
- note removed: "SWD Interface"
- note removed: "USB Entry"
- note removed: "USB Interface"
- moved on the sheet: H1, H2, Q1, R1, R2, R3

Commit message: Finished mainboard schematic layout
Parts:
- removed J? (x3): Conn_01x04, symbol Connector:Conn_01x04_Male
- added J12, J13, J7: 0530470310, Connector_Molex:Molex_PicoBlade_53047-0310_1x03_P1.25mm_Vertical, symbol Connector:Conn_01x03_Male
- added J14: Conn_02x04_Odd_Even, Connector_PinHeader_2.54mm:PinHeader_2x04_P2.54mm_Vertical, symbol Connector_Generic:Conn_02x04_Odd_Even
- added J16, J5, J8: Conn_01x04_Male, Connector_PinHeader_2.54mm:PinHeader_1x04_P2.54mm_Vertical, symbol Connector:Conn_01x04_Male
- added R4, R5, R6, R7: 15k, Resistor_SMD:R_1206_3216Metric, symbol Device:R_Small_US
- J1, J2, J4: renamed from J?; value Conn_01x02_Male -> 0530470210; footprint (none) -> Connector_Molex:Molex_PicoBlade_53047-0210_1x02_P1.25mm_Vertical
- J10, J15, J3: renamed from J?; value Conn_01x03_Male -> 0530470310; footprint (none) -> Connector_Molex:Molex_PicoBlade_53047-0310_1x03_P1.25mm_Vertical
- J11, J9: renamed from J?; value Conn_01x04 -> 0530470410; footprint (none) -> Connector_Molex:Molex_PicoBlade_53047-0410_1x04_P1.25mm_Vertical
- J17: renamed from J?; footprint (none) -> Connector_PinSocket_2.54mm:PinSocket_2x20_P2.54mm_Vertical
- J6: renamed from J?; value Conn_01x04 -> 0530470310; footprint (none) -> Connector_Molex:Molex_PicoBlade_53047-0310_1x03_P1.25mm_Vertical; symbol Connector:Conn_01x04_Male -> Connector:Conn_01x03_Male
- gave numbers to parts that had none: 2
Connections:
- net +3V3: now also J16.1 (Pin_1), J5.1 (Pin_1), J8.1 (Pin_1), R4.1, R5.1, R6.1, R7.1; no longer J6.2 (Pin_2)
- net +5V: now also J12.1 (Pin_1), J13.1 (Pin_1), J7.1 (Pin_1)
- net BUZZER: now also J17.32 (PWM0/GPIO12)
- net GND: now also J6.3 (Pin_3), J12.3 (Pin_3), J13.3 (Pin_3), J14.2 (Pin_2), J14.4 (Pin_4), J14.6 (Pin_6), J14.8 (Pin_8), J16.4 (Pin_4), J5.4 (Pin_4), J7.3 (Pin_3), J8.4 (Pin_4); no longer J6.4 (Pin_4)
- net MUTE: now also J17.13 (GPIO27), J16.2 (Pin_2)
- net UI_BUTTON: now also J17.15 (GPIO22), J16.3 (Pin_3)
- net LED0_SDO: now reaches J9.2 (Pin_2)
- net LED0_SDO: now also J17.21 (MISO0/GPIO9), J5.2 (Pin_2)
- net LED0_SCK: now reaches J9.3 (Pin_3)
- net LED0_SCK: now also J17.23 (SCLK0/GPIO11), J5.3 (Pin_3)
- net EXP1: now reaches J17.11 (GPIO17)
- net EXP1: now also J15.2 (Pin_2)
- net PROX1_OUT: now reaches J17.29 (GCLK1/GPIO5)
- net PROX1_OUT: now also J6.2 (Pin_2), J14.1 (Pin_1), R4.2
- net PROX2_OUT: now reaches J17.31 (GCLK2/GPIO6)
- net PROX2_OUT: now also J12.2 (Pin_2), J14.3 (Pin_3), R6.2
- net PROX3_OUT: now reaches J17.33 (PWM1/GPIO13)
- net PROX3_OUT: now also J14.5 (Pin_5), J7.2 (Pin_2), R5.2
- net LED1_SDO: now reaches J17.35 (GPIO19/MISO1)
- net LED1_SDO: now also J11.2 (Pin_2), J8.2 (Pin_2)
- net EXP0: now reaches J17.36 (GPIO16)
- net EXP0: now also J10.2 (Pin_2)
- net PROX4_OUT: now reaches J17.37 (GPIO26)
- net PROX4_OUT: now also J13.2 (Pin_2), J14.7 (Pin_7), R7.2
- net LED1_SCK: now reaches J17.40 (GPIO21/SCLK1)
- net LED1_SCK: now also J11.3 (Pin_3), J8.3 (Pin_3)
- no-connect marks 0 -> 15
Other:
- note added: "Debug Headers"
- note added: "LED Conn."
- note added: "Prox Sensor"
- note added: "UI Buttons"
- note removed: "Panel Mount"
- moved on the sheet: H1, H2, H3, H4, J1, J10, J11, J15, J17, J2, J3, J4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

Commit message: Finished mainboard pcb routing
Parts:
- removed J2: 0530470210, Connector_Molex:Molex_PicoBlade_53047-0210_1x02_P1.25mm_Vertical, symbol Connector:Conn_01x02_Male
- J16: value Conn_01x04_Male -> Conn_01x03_Male; footprint Connector_PinHeader_2.54mm:PinHeader_1x04_P2.54mm_Vertical -> Connector_PinHeader_2.54mm:PinHeader_1x03_P2.54mm_Vertical; symbol Connector:Conn_01x04_Male -> Connector:Conn_01x03_Male
Connections:
- net +3V3: no longer J16.1 (Pin_1), J17.17 (3V3)
- net GND: now also J16.3 (Pin_3); no longer J16.4 (Pin_4), J17.14 (GND), J17.20 (GND), J17.25 (GND), J17.39 (GND), J17.9 (GND)
- net MUTE: now also J16.1 (Pin_1); no longer J16.2 (Pin_2)
- net UI_BUTTON: now also J16.2 (Pin_2); no longer J16.3 (Pin_3)
- no-connect marks 15 -> 22
Other:
- note removed: "5V Entry"
- moved on the sheet: J14, J5, J8

Commit message: Changed pin assignments for cleaner PCB routing
Parts:
- J5, J8: value Conn_01x04_Male -> Conn_01x03_Male; footprint Connector_PinHeader_2.54mm:PinHeader_1x04_P2.54mm_Vertical -> Connector_PinHeader_2.54mm:PinHeader_1x03_P2.54mm_Vertical; symbol Connector:Conn_01x04_Male -> Connector:Conn_01x03_Male
Connections:
- net +3V3: now also J17.17 (3V3); no longer J5.1 (Pin_1), J8.1 (Pin_1)
- net BUZZER: now also J17.33 (PWM1/GPIO13); no longer J17.32 (PWM0/GPIO12)
- net EXP0: now also J17.10 (GPIO15/RXD); no longer J17.36 (GPIO16)
- net EXP1: now also J17.8 (GPIO14/TXD); no longer J17.11 (GPIO17)
- net GND: now also J17.14 (GND), J17.20 (GND), J17.25 (GND), J17.39 (GND), J17.9 (GND), J5.3 (Pin_3), J8.3 (Pin_3); no longer J5.4 (Pin_4), J8.4 (Pin_4)
- net LED0_SCK: now also J5.2 (Pin_2); no longer J5.3 (Pin_3)
- net LED0_SDO: now also J5.1 (Pin_1); no longer J5.2 (Pin_2)
- net LED1_SCK: now also J8.2 (Pin_2); no longer J8.3 (Pin_3)
- net LED1_SDO: now also J8.1 (Pin_1); no longer J8.2 (Pin_2)
- net MUTE: now also J17.31 (GCLK2/GPIO6); no longer J17.13 (GPIO27)
- net PROX1_OUT: now also J12.2 (Pin_2), J14.3 (Pin_3), J17.11 (GPIO17), R6.2; no longer J14.1 (Pin_1), J17.29 (GCLK1/GPIO5), J6.2 (Pin_2), R4.2
- net PROX2_OUT: now also J14.5 (Pin_5), J17.13 (GPIO27), J7.2 (Pin_2), R5.2; no longer J12.2 (Pin_2), J14.3 (Pin_3), J17.31 (GCLK2/GPIO6), R6.2
- net PROX3_OUT: now also J13.2 (Pin_2), J14.7 (Pin_7), J17.15 (GPIO22), R7.2; no longer J14.5 (Pin_5), J17.33 (PWM1/GPIO13), J7.2 (Pin_2), R5.2
- net UI_BUTTON: now also J17.29 (GCLK1/GPIO5); no longer J17.15 (GPIO22)
- net PROX0_OUT: now reaches J17.7 (GCLK0/GPIO4)
- net PROX0_OUT: now also J14.1 (Pin_1), J6.2 (Pin_2), R4.2
- removed net PROX4_OUT: J13.2 (Pin_2), J14.7 (Pin_7), J17.37 (GPIO26), R7.2
- no-connect marks 22 -> 15
Other:
- moved on the sheet: J11, J9
