File: ecad/reminder-mainboard/reminder-mainboard.sch (KiCad schematic (older format))
At the start: 28 parts, among them J1 0530470210, J10 0530470310, J11 0530470410, J12 0530470310, J13 0530470310, J14 Conn_02x04_Odd_Even, J15 0530470310, J16 Conn_01x03_Male, J17 Raspberry_Pi_2_3, J3 0530470310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

Commit message: Added LCSC part numbers, minor tweaks based on part availablity.
Parts:
- removed J5: Conn_01x03_Male, Connector_PinHeader_2.54mm:PinHeader_1x03_P2.54mm_Vertical, symbol Connector:Conn_01x03_Male
- added C1: 100uf, Capacitor_Tantalum_SMD:CP_EIA-3528-21_Kemet-B, symbol Device:C_Small
- added D1: 19-217/BHC-ZL1M2RY/3T, LED_SMD:LED_0603_1608Metric, symbol Device:LED
- added J2: 0530470210, Connector_Molex:Molex_PicoBlade_53047-0210_1x02_P1.25mm_Vertical, symbol Connector:Conn_01x02_Male
- added R8: 120, Resistor_SMD:R_0603_1608Metric, symbol Device:R_Small_US
- H1, H2, H3, H4: footprint MountingHole:MountingHole_2.7mm_M2.5_Pad -> MountingHole:MountingHole_2.7mm_M2.5; DNP (none) -> 1
- J1, J10, J11, J12, J13, J14, J15, J16, J17, J3, J4, J6, J7, J9: DNP (none) -> 1
- J8: value Conn_01x03_Male -> Conn_02x03_Male; footprint Connector_PinHeader_2.54mm:PinHeader_1x03_P2.54mm_Vertical -> Connector_PinHeader_2.54mm:PinHeader_2x03_P2.54mm_Vertical; symbol Connector:Conn_01x03_Male -> Connector_Generic:Conn_02x03_Odd_Even; DNP (none) -> 1
- Q1: value 2N3904 -> S9013; symbol Transistor_BJT:2N3904 -> Device:Q_NPN_BEC; LCSC Part Number (none) -> C6749; Mfg PN S8050 -> (none)
- R1: value 510 -> 2.2k; LCSC Part Number (none) -> C4190; Mfg Uniroyal Elec -> (none); Mfg PN 0603WAF5100T5E -> (none)
- R2, R3: value 10k -> 11k; LCSC Part Number (none) -> C25950; Mfg Uniroyal Elec -> (none); Mfg PN 0603WAF1002T5E -> (none)
- R4, R5, R6, R7: value 15k -> 10k; LCSC Part Number (none) -> C17902
Connections:
- net +5V: now also C1.1, J2.1 (Pin_1), R8.1
- net GND: now also J8.5 (Pin_5), J8.6 (Pin_6), Q1.2 (E), C1.2, D1.1 (K), J2.2 (Pin_2); no longer J8.3 (Pin_3), Q1.1 (E)
- net LED0_SCK: now also J8.3 (Pin_3)
- net LED0_SDO: now also J8.1 (Pin_1)
- net LED1_SCK: now also J8.4 (Pin_4); no longer J8.2 (Pin_2)
- net LED1_SDO: now also J8.2 (Pin_2); no longer J8.1 (Pin_1)
- net at R1.2: now also Q1.1 (B); no longer Q1.2 (B)
- new net: D1.2 (A), R8.2
Other:
- note added: "5V In"
- note added: "Raspberry Pi Zero Header"
- moved on the sheet: H1, H2, H3, H4, J17

Commit message: Created production files and gerbers
Parts:
- C1: LCSC (none) -> C16133
- D1: LCSC (none) -> C72041
- Q1: LCSC (none) -> C6749
- R1: LCSC (none) -> C4190
- R2, R3: LCSC (none) -> C25950
- R4, R5, R6, R7: LCSC (none) -> C17902
- R8: LCSC (none) -> C22787
Changed lines of the file:
@@
 F 5 "" H 1600 5300 50  0001 C CNN "Mfg PN"
 F 6 "C25950" H 1600 5300 50  0001 C CNN "LCSC Part Number"
+F 7 "C25950" H 1600 5300 50  0001 C CNN "LCSC"
 	1    1600 5300
 	1    0    0    -1
@@
 F 5 "" H 1500 1350 50  0001 C CNN "Mfg PN"
 F 6 "C25950" H 1500 1350 50  0001 C CNN "LCSC Part Number"
+F 7 "C25950" H 1500 1350 50  0001 C CNN "LCSC"
 	1    1500 1350
 	1    0    0    -1
@@
 F 5 "" H 1100 1800 50  0001 C CNN "Mfg PN"
 F 6 "C4190" H 1100 1800 50  0001 C CNN "LCSC Part Number"
+F 7 "C4190" H 1100 1800 50  0001 C CNN "LCSC"
 	1    1100 1800
 	0    -1   -1   0
@@
 F 5 "" H 1550 1800 50  0001 C CNN "Mfg PN"
 F 6 "C6749" H 1550 1800 50  0001 C CNN "LCSC Part Number"
+F 7 "C6749" H 1550 1800 50  0001 C CNN "LCSC"
 	1    1550 1800
 	1    0    0    -1
@@
 F 3 "~" H 4200 5200 50  0001 C CNN
 F 4 "C17902" H 4200 5200 50  0001 C CNN "LCSC Part Number"
+F 5 "C17902" H 4200 5200 50  0001 C CNN "LCSC"
 	1    4200 5200
 	1    0    0    -1
@@
 F 3 "~" H 6050 5200 50  0001 C CNN
 F 4 "C17902" H 6050 5200 50  0001 C CNN "LCSC Part Number"
+F 5 "C17902" H 6050 5200 50  0001 C CNN "LCSC"
 	1    6050 5200
 	1    0    0    -1
@@
 F 3 "~" H 6050 4250 50  0001 C CNN
 F 4 "C17902" H 6050 4250 50  0001 C CNN "LCSC Part Number"
+F 5 "C17902" H 6050 4250 50  0001 C CNN "LCSC"
 	1    6050 4250
 	1    0    0    -1
@@
 F 3 "~" H 4200 4250 50  0001 C CNN
 F 4 "C17902" H 4200 4250 50  0001 C CNN "LCSC Part Number"
+F 5 "C17902" H 4200 4250 50  0001 C CNN "LCSC"
 	1    4200 4250
 	1    0    0    -1
@@
 F 3 "~" H 8300 1200 50  0001 C CNN
 F 4 "C22787" H 8300 1200 50  0001 C CNN "LCSC Part Number"
+F 5 "C22787" H 8300 1200 50  0001 C CNN "LCSC"
 	1    8300 1200
 	1    0    0    -1
@@
 F 3 "~" H 8300 1450 50  0001 C CNN
 F 4 "C72041" H 8300 1450 50  0001 C CNN "LCSC Part Number"
+F 5 "C72041" H 8300 1450 50  0001 C CNN "LCSC"
 	1    8300 1450
 	0    -1   -1   0
@@
 F 3 "~" H 7800 1150 50  0001 C CNN
 F 4 "C16133" H 7800 1150 50  0001 C CNN "LCSC Part Number"
+F 5 "C16133" H 7800 1150 50  0001 C CNN "LCSC"
 	1    7800 1150
 	1    0    0    -1
